File: 4 GC port esd board (for wii mini)/4 GC port esd board (for wii mini).kicad_pcb (KiCad board)
At the start: 2 copper layers, 17.5 x 46 mm, 20 parts, among them J1 port 4, J2 port 1, J3 port 2, J4 port 3, J5 power, J6 controller ports

Commit message: updated silk
Parts:
- moved G*** 6.76 mm to (110.2, 75.2)
- moved G*** 6.20 mm to (110.2, 103.1)
Other:
- board text added: "3.3v"
- board text added: "Dat"
Changed lines of the file:
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@@
   )
   (footprint "Evan's misc parts:OSHW gear" (layer "B.Cu")
-    (at 106.426 69.596 -90)
+    (at 110.236 75.184 -90)
     (attr board_only exclude_from_pos_files exclude_from_bom)
     (fp_text reference "G***" (at 0 -5.08 90) (layer "B.Fab") hide
@@
   )
   (footprint "Evan's misc parts:Evan Logo" (layer "B.Cu")
-    (at 106.68 108.204 -90)
+    (at 110.236 103.124 -90)
     (attr board_only exclude_from_pos_files exclude_from_bom)
     (fp_text reference "G***" (at 0.397791 -5.08 90) (layer "B.Fab") hide
@@
   (gr_line (start 99.06 112.014) (end 99.06 111.252) (layer "Edge.Cuts") (width 0.1))
   (gr_line (start 100.33 66.04) (end 99.06 66.04) (layer "Edge.Cuts") (width 0.1))
-  (gr_text "wii mini controller esd board" (at 110.49 85.852 90) (layer "B.SilkS")
+  (gr_text "Dat" (at 104.902 96.266) (layer "B.SilkS")
     (effects (font (size 1 1) (thickness 0.15)) (justify mirror))
   )
-  (gr_text "abzman2k.wordpress.com" (at 104.902 96.52 90) (layer "B.SilkS")
+  (gr_text "Gnd" (at 104.902 82.296) (layer "B.SilkS")
     (effects (font (size 1 1) (thickness 0.15)) (justify mirror))
   )
+  (gr_text "wii mini controller esd board" (at 110.744 88.9 90) (layer "B.SilkS")
+    (effects (font (size 1 1) (thickness 0.15)) (justify mirror))
+  )
+  (gr_text "5v" (at 104.648 79.756) (layer "B.SilkS")
+    (effects (font (size 1 1) (thickness 0.15)) (justify mirror))
+  )
+  (gr_text "Gnd" (at 104.902 93.726) (layer "B.SilkS")
+    (effects (font (size 1 1) (thickness 0.15)) (justify mirror))
+  )
+  (gr_text "3.3v" (at 105.156 98.806) (layer "B.SilkS")
+    (effects (font (size 1 1) (thickness 0.15)) (justify mirror))
+  )
+  (gr_text "Gnd" (at 104.902 70.612) (layer "B.SilkS")
+    (effects (font (size 1 1) (thickness 0.15)) (justify mirror))
+  )
+  (gr_text "Dat" (at 105.156 84.836) (layer "B.SilkS")
+    (effects (font (size 1 1) (thickness 0.15)) (justify mirror))
+  )
+  (gr_text "abzman2k.wordpress.com" (at 109.22 90.932 90) (layer "B.SilkS")
+    (effects (font (size 1 1) (thickness 0.15)) (justify mirror))
+  )
+  (gr_text "5v" (at 104.648 91.44) (layer "B.SilkS")
+    (effects (font (size 1 1) (thickness 0.15)) (justify mirror))
+  )
+  (gr_text "Dat" (at 105.156 73.152) (layer "B.SilkS")
+    (effects (font (size 1 1) (thickness 0.15)) (justify mirror))
+  )
+  (gr_text "Dat" (at 104.902 107.696) (layer "B.SilkS")
+    (effects (font (size 1 1) (thickness 0.15)) (justify mirror))
+  )
+  (gr_text "5v" (at 104.648 68.072) (layer "B.SilkS")
+    (effects (font (size 1 1) (thickness 0.15)) (justify mirror))
+  )
+  (gr_text "3.3v" (at 105.156 87.376) (layer "B.SilkS")
+    (effects (font (size 1 1) (thickness 0.15)) (justify mirror))
+  )
+  (gr_text "3.3v" (at 105.156 110.236) (layer "B.SilkS")
+    (effects (font (size 1 1) (thickness 0.15)) (justify mirror))
+  )
+  (gr_text "Gnd" (at 104.902 105.156) (layer "B.SilkS")
+    (effects (font (size 1 1) (thickness 0.15)) (justify mirror))
+  )
+  (gr_text "3.3v" (at 105.156 75.692) (layer "B.SilkS")
+    (effects (font (size 1 1) (thickness 0.15)) (justify mirror))
+  )
+  (gr_text "5v" (at 104.648 102.616) (layer "B.SilkS")
+    (effects (font (size 1 1) (thickness 0.15)) (justify mirror))
+  )
